Commit message: adjusted disk paras, added contacting constrain

File: assets/objects/disk/disk.urdf (robot description, URDF)
Before this commit: robot disk.urdf, 1 links, 0 joints
Links:
- link baseLink: mass 5. -> 3.; geometry collision cylinder length=0.04 radius=0.06; visual cylinder length=0.04 radius=0.06

Commit message: renamed obejects, finished model training

File: assets/objects/disk/disk.urdf (robot description, URDF)
Before this commit: robot disk.urdf, 1 links, 0 joints
Links:
- link baseLink: mass 3. -> 2.5

Commit message: added dims to state and added angle to loss, increase success rate to 50%

File: assets/objects/disk/disk.urdf (robot description, URDF)
Before this commit: robot disk.urdf, 1 links, 0 joints
Links:
- link baseLink: mass 2.5 -> 1.5
